File: file5F9EC5F3.sch (KiCad schematic (older format))
At the start: 1 part

Commit message: Cosas
- Power
- I/O
- Screen
- Sensing
Parts:
- added J4: Conn_ARM_JTAG_SWD_10, symbol Connector:Conn_ARM_JTAG_SWD_10
- gave numbers to parts that had none: 1
Connections:
- new net +3V3: J4.1 (VTref)
- new net GND: J4.3 (GND), J4.5 (GND)
- new net RST: J4.10 (~RESET~)
Changed lines of the file:
@@
 $Descr A4 11693 8268
 encoding utf-8
-Sheet 2 4
+Sheet 7 7
 Title ""
 Date ""
@@
 $EndDescr
 $Comp
-L MCU_ST_STM32F1:STM32F102C8Tx U?
+L MCU_ST_STM32F1:STM32F102C8Tx U3
 U 1 1 5F9EEC89
 P 6000 3650
-F 0 "U?" H 5950 2061 50  0000 C CNN
+F 0 "U3" H 5950 2061 50  0000 C CNN
 F 1 "STM32F102C8Tx" H 5950 1970 50  0000 C CNN
 F 2 "Package_QFP:LQFP-48_7x7mm_P0.5mm" H 5400 2250 50  0001 R CNN
@@
 Wire Wire Line
 	5300 2850 4950 2850
+Text HLabel 4450 4650 0    50   Output ~ 0
+PELTIER_EN_1
+Text HLabel 4450 3950 0    50   Output ~ 0
+PELTIER_EN_2
+Text HLabel 4450 4050 0    50   Output ~ 0
+PELTIER_IN_A_2
+Text HLabel 4450 4550 0    50   Output ~ 0
+PELTIER_IN_A_1
+Text HLabel 4450 4150 0    50   Output ~ 0
+PELTIER_IN_B_2
+Text HLabel 4450 4450 0    50   Output ~ 0
+PELTIER_IN_B_1
+Text HLabel 4450 4250 0    50   Output ~ 0
+PELTIER_PWM_2
+Text HLabel 4450 4750 0    50   Output ~ 0
+PELTIER_PWM_1
+Text HLabel 7650 3500 2    50   Output ~ 0
+SCREEN_D-C_SPI
+Text HLabel 7650 3600 2    50   Output ~ 0
+SCREEN_CS_SPI
+Text HLabel 7650 3700 2    50   Output ~ 0
+SCREEN_RESET
+Text HLabel 7650 3800 2    50   Output ~ 0
+SD_CS_SPI
+Text HLabel 7650 3900 2    50   Output ~ 0
+SD_FLASH
+Text HLabel 7650 4000 2    50   Output ~ 0
+MISO_OUT
+Text HLabel 7650 4100 2    50   Output ~ 0
+MOSI_OUT
+Text HLabel 7650 4200 2    50   Output ~ 0
+SPI_CLOCK_IN
+Text HLabel 7650 4300 2    50   Output ~ 0
+BUZZER_PWM_IN
+Text HLabel 7650 4500 2    50   Input ~ 0
+THERMISTOR_IN_1
+Text HLabel 7650 4600 2    50   Input ~ 0
+THERMISTOR_IN_2
+Text HLabel 7650 4750 2    50   Input ~ 0
+BT_STATE
+Text HLabel 7650 4850 2    50   Output ~ 0
+BT_RXD
+Text HLabel 7650 4950 2    50   Input ~ 0
+BT_TXD
+Text HLabel 7650 5050 2    50   Output ~ 0
+BT_ENABLE
+Text HLabel 7650 5150 2    50   BiDi ~ 0
+USB_DATA_MINUS
+Text HLabel 7650 5250 2    50   BiDi ~ 0
+USB_DATA_PLUS
+$Comp
+L Connector:Conn_ARM_JTAG_SWD_10 J4
+U 1 1 5FA20544
+P 2850 1450
+F 0 "J4" H 2407 1496 50  0000 R CNN
+F 1 "Conn_ARM_JTAG_SWD_10" H 2407 1405 50  0000 R CNN
+F 2 "" H 2850 1450 50  0001 C CNN
+F 3 "http://infocenter.arm.com/help/topic/com.arm.doc.ddi0314h/DDI0314H_coresight_components_trm.pdf" V 2500 200 50  0001 C CNN
+	1    2850 1450
+	1    0    0    -1
+$EndComp
+$Comp
+L power:GND #PWR016
+U 1 1 5FA20D76
+P 2850 2250
+F 0 "#PWR016" H 2850 2000 50  0001 C CNN
+F 1 "GND" H 2855 2077 50  0000 C CNN
+F 2 "" H 2850 2250 50  0001 C CNN
+F 3 "" H 2850 2250 50  0001 C CNN
+	1    2850 2250
+	1    0    0    -1
+$EndComp
+Wire Wire Line
+	2850 2050 2850 2250
+$Comp
+L power:+3.3V #PWR015
+U 1 1 5FA21240
+P 2850 700
+F 0 "#PWR015" H 2850 550 50  0001 C CNN
+F 1 "+3.3V" H 2865 873 50  0000 C CNN
+F 2 "" H 2850 700 50  0001 C CNN
+F 3 "" H 2850 700 50  0001 C CNN
+	1    2850 700
+	1    0    0    -1
+$EndComp
+Wire Wire Line
+	2850 700  2850 850
+Text Label 3750 1150 0    50   ~ 0
+RST
+Wire Wire Line
+	3750 1150 3350 1150
 $EndSCHEMATC

Commit message: Finished schematic
Parts:
- removed U3: STM32F102C8Tx, Package_QFP:LQFP-48_7x7mm_P0.5mm, symbol MCU_ST_STM32F1:STM32F102C8Tx
- added C1, C10, C11, C2, C3, C4, C5, C7, C8, C9: 100nF, symbol Device:C
- added C6: C, symbol Device:C
- added R10, R9: 390, symbol Device:R
- added R6, R8: 10k, symbol Device:R
- added SW1: SW_Push, symbol Switch:SW_Push
- added SW2, SW3: SW_SPDT, symbol Switch:SW_SPDT
- added U3: STM32F102R8Tx, Package_QFP:LQFP-64_10x10mm_P0.5mm, symbol MCU_ST_STM32F1:STM32F102R8Tx
- added Y1: 32KHz, symbol Device:Crystal
- added Y2: 8MHz, symbol Device:Crystal
Connections:
- net +3V3: now also C10.1, C11.1, C5.1, C7.1, C8.1, C9.1, U3.1 (VBAT), U3.13 (VDDA), U3.19 (VDD), U3.32 (VDD), U3.48 (VDD), U3.64 (VDD)
- net BT_ENABLE: now also U3.14 (PA0)
- net BT_RXD: now also U3.15 (PA1)
- net BT_STATE: now also U3.17 (PA3)
- net BT_TXD: now also U3.16 (PA2)
- net BUZZER_PWM_IN: now also U3.26 (PB0)
- net GND: now also C1.2, C10.2, C11.2, C2.2, C3.2, C4.2, C5.2, C6.2, C7.2, C8.2, C9.2, SW1.2, SW2.3 (C), SW3.3 (C), U3.12 (VSSA), U3.18 (VSS), U3.31 (VSS), U3.47 (VSS), U3.63 (VSS)
- net MISO_OUT: now also U3.35 (PB14)
- net MOSI_OUT: now also U3.36 (PB15)
- net PELTIER_EN_1: now also U3.57 (PB5)
- net PELTIER_EN_2: now also U3.51 (PC10)
- net PELTIER_IN_A_1: now also U3.58 (PB6)
- net PELTIER_IN_A_2: now also U3.52 (PC11)
- net PELTIER_IN_B_1: now also U3.59 (PB7)
- net PELTIER_IN_B_2: now also U3.53 (PC12)
- net PELTIER_PWM_1: now also U3.61 (PB8)
- net PELTIER_PWM_2: now also U3.54 (PD2)
- net RST: now also C6.1, SW1.1, U3.7 (NRST)
- net SCREEN_CS_SPI: now also U3.33 (PB12)
- net SCREEN_D-C_SPI: now also U3.38 (PC7)
- net SCREEN_RESET: now also U3.39 (PC8)
- net SD_CS_SPI: now also U3.41 (PA8)
- net SD_FLASH: now also U3.42 (PA9)
- net SPI_CLOCK_IN: now also U3.34 (PB13)
- net THERMISTOR_IN_1: now also U3.24 (PC4)
- net THERMISTOR_IN_2: now also U3.25 (PC5)
- net USB_DATA_MINUS: now also U3.43 (PA10)
- net USB_DATA_PLUS: now also U3.44 (PA11)
- net SWDIO: now reaches J4.2 (SWDIO/TMS)
- net SWDIO: now also U3.46 (PA13)
- net SWDCLK: now reaches J4.4 (SWDCLK/TCK)
- net SWDCLK: now also U3.49 (PA14)
- net SWO: now reaches J4.6 (SWO/TDO)
- net SWO: now also U3.55 (PB3)
- net JTDI: now reaches J4.8 (NC/TDI)
- net JTDI: now also U3.50 (PA15)
- new net: R6.1, SW2.2 (B)
- new net: R8.1, SW3.2 (B)
- new net: C4.1, R10.2, Y2.2
- new net: C2.1, R9.2, Y1.2
- new net +5V: SW2.1 (A), SW3.1 (A)
- new net BOOT0: R8.2, U3.60 (BOOT0)
- new net BOOT1: R6.2, U3.28 (PB2)
- new net OSC_IN_HSE: C3.1, U3.5 (PD0), Y2.1
- new net OSC_IN_LSE: C1.1, U3.3 (PC14), Y1.1
- new net OSC_OUT_HSE: R10.1, U3.6 (PD1)
- new net OSC_OUT_LSE: R9.1, U3.4 (PC15)
- no-connect marks 0 -> 13
Other:
- moved on the sheet: J4

Commit message: Added footprints
Parts:
- C1, C10, C11, C2, C3, C4, C5, C7, C8, C9: footprint (none) -> Capacitor_SMD:C_0805_2012Metric
- C6: value C -> 100nf; footprint (none) -> Capacitor_SMD:C_0805_2012Metric
- J4: footprint (none) -> Connector_JST:JST_EH_B10B-EH-A_1x10_P2.50mm_Vertical
- R10, R6, R8, R9: footprint (none) -> Resistor_SMD:R_0805_2012Metric
- SW1: footprint (none) -> Button_Switch_SMD:SW_SPST_CK_RS282G05A3
- SW2, SW3: footprint (none) -> Button_Switch_SMD:SW_SPDT_PCM12
- Y1, Y2: footprint (none) -> Crystal:Resonator-2Pin_W7.0mm_H2.5mm
Changed lines of the file:
@@
 F 0 "J4" H 2207 1646 50  0000 R CNN
 F 1 "Conn_ARM_JTAG_SWD_10" H 2207 1555 50  0000 R CNN
-F 2 "" H 2650 1600 50  0001 C CNN
+F 2 "Connector_JST:JST_EH_B10B-EH-A_1x10_P2.50mm_Vertical" H 2650 1600 50  0001 C CNN
 F 3 "http://infocenter.arm.com/help/topic/com.arm.doc.ddi0314h/DDI0314H_coresight_components_trm.pdf" V 2300 350 50  0001 C CNN
 	1    2650 1600
@@
 F 0 "R6" V 1093 7100 50  0000 C CNN
 F 1 "10k" V 1184 7100 50  0000 C CNN
-F 2 "" V 1230 7100 50  0001 C CNN
+F 2 "Resistor_SMD:R_0805_2012Metric" V 1230 7100 50  0001 C CNN
 F 3 "~" H 1300 7100 50  0001 C CNN
 	1    1300 7100
@@
 F 0 "C5" H 9865 1146 50  0000 L CNN
 F 1 "100nF" H 9865 1055 50  0000 L CNN
-F 2 "" H 9788 950 50  0001 C CNN
+F 2 "Capacitor_SMD:C_0805_2012Metric" H 9788 950 50  0001 C CNN
 F 3 "~" H 9750 1100 50  0001 C CNN
 	1    9750 1100
@@
 F 0 "SW2" H 1650 7385 50  0000 C CNN
 F 1 "SW_SPDT" H 1650 7294 50  0000 C CNN
-F 2 "" H 1650 7100 50  0001 C CNN
+F 2 "Button_Switch_SMD:SW_SPDT_PCM12" H 1650 7100 50  0001 C CNN
 F 3 "~" H 1650 7100 50  0001 C CNN
 	1    1650 7100
@@
 F 0 "R8" V 1143 5950 50  0000 C CNN
 F 1 "10k" V 1234 5950 50  0000 C CNN
-F 2 "" V 1280 5950 50  0001 C CNN
+F 2 "Resistor_SMD:R_0805_2012Metric" V 1280 5950 50  0001 C CNN
 F 3 "~" H 1350 5950 50  0001 C CNN
 	1    1350 5950
@@
 F 0 "SW3" H 1700 6235 50  0000 C CNN
 F 1 "SW_SPDT" H 1700 6144 50  0000 C CNN
-F 2 "" H 1700 5950 50  0001 C CNN
+F 2 "Button_Switch_SMD:SW_SPDT_PCM12" H 1700 5950 50  0001 C CNN
 F 3 "~" H 1700 5950 50  0001 C CNN
 	1    1700 5950
@@
 F 0 "SW1" H 1700 4935 50  0000 C CNN
 F 1 "SW_Push" H 1700 4844 50  0000 C CNN
-F 2 "" H 1700 4850 50  0001 C CNN
+F 2 "Button_Switch_SMD:SW_SPST_CK_RS282G05A3" H 1700 4850 50  0001 C CNN
 F 3 "~" H 1700 4850 50  0001 C CNN
 	1    1700 4650
@@
 F 0 "Y2" V 4204 7231 50  0000 L CNN
 F 1 "8MHz" V 4295 7231 50  0000 L CNN
-F 2 "" H 4250 7100 50  0001 C CNN
+F 2 "Crystal:Resonator-2Pin_W7.0mm_H2.5mm" H 4250 7100 50  0001 C CNN
 F 3 "~" H 4250 7100 50  0001 C CNN
 	1    4250 7100
@@
 F 0 "C3" V 3650 6850 50  0000 C CNN
 F 1 "100nF" V 3739 6950 50  0000 C CNN
-F 2 "" H 3938 6800 50  0001 C CNN
+F 2 "Capacitor_SMD:C_0805_2012Metric" H 3938 6800 50  0001 C CNN
 F 3 "~" H 3900 6950 50  0001 C CNN
 	1    3900 6950
@@
 F 0 "C4" V 4150 7150 50  0000 C CNN
 F 1 "100nF" V 4050 7250 50  0000 C CNN
-F 2 "" H 3938 7100 50  0001 C CNN
+F 2 "Capacitor_SMD:C_0805_2012Metric" H 3938 7100 50  0001 C CNN
 F 3 "~" H 3900 7250 50  0001 C CNN
 	1    3900 7250
@@
 F 0 "C1" V 3600 5650 50  0000 C CNN
 F 1 "100nF" V 3689 5750 50  0000 C CNN
-F 2 "" H 3888 5600 50  0001 C CNN
+F 2 "Capacitor_SMD:C_0805_2012Metric" H 3888 5600 50  0001 C CNN
 F 3 "~" H 3850 5750 50  0001 C CNN
 	1    3850 5750
@@
 F 0 "C2" V 4100 5950 50  0000 C CNN
 F 1 "100nF" V 4000 6050 50  0000 C CNN
-F 2 "" H 3888 5900 50  0001 C CNN
+F 2 "Capacitor_SMD:C_0805_2012Metric" H 3888 5900 50  0001 C CNN
 F 3 "~" H 3850 6050 50  0001 C CNN
 	1    3850 6050
@@
 F 0 "Y1" V 4154 6031 50  0000 L CNN
 F 1 "32KHz" V 4245 6031 50  0000 L CNN
-F 2 "" H 4200 5900 50  0001 C CNN
+F 2 "Crystal:Resonator-2Pin_W7.0mm_H2.5mm" H 4200 5900 50  0001 C CNN
 F 3 "~" H 4200 5900 50  0001 C CNN
 	1    4200 5900
@@
 F 0 "R9" V 4593 6050 50  0000 C CNN
 F 1 "390" V 4684 6050 50  0000 C CNN
-F 2 "" V 4730 6050 50  0001 C CNN
+F 2 "Resistor_SMD:R_0805_2012Metric" V 4730 6050 50  0001 C CNN
 F 3 "~" H 4800 6050 50  0001 C CNN
 	1    4800 6050
@@
 F 0 "R10" V 4593 7250 50  0000 C CNN
 F 1 "390" V 4684 7250 50  0000 C CNN
-F 2 "" V 4730 7250 50  0001 C CNN
+F 2 "Resistor_SMD:R_0805_2012Metric" V 4730 7250 50  0001 C CNN
 F 3 "~" H 4800 7250 50  0001 C CNN
 	1    4800 7250
@@
 F 0 "C9" H 9365 1146 50  0000 L CNN
 F 1 "100nF" H 9365 1055 50  0000 L CNN
-F 2 "" H 9288 950 50  0001 C CNN
+F 2 "Capacitor_SMD:C_0805_2012Metric" H 9288 950 50  0001 C CNN
 F 3 "~" H 9250 1100 50  0001 C CNN
 	1    9250 1100
@@
 F 0 "C8" H 8865 1146 50  0000 L CNN
 F 1 "100nF" H 8865 1055 50  0000 L CNN
-F 2 "" H 8788 950 50  0001 C CNN
+F 2 "Capacitor_SMD:C_0805_2012Metric" H 8788 950 50  0001 C CNN
 F 3 "~" H 8750 1100 50  0001 C CNN
 	1    8750 1100
@@
 F 0 "C10" H 10365 1146 50  0000 L CNN
 F 1 "100nF" H 10365 1055 50  0000 L CNN
-F 2 "" H 10288 950 50  0001 C CNN
+F 2 "Capacitor_SMD:C_0805_2012Metric" H 10288 950 50  0001 C CNN
 F 3 "~" H 10250 1100 50  0001 C CNN
 	1    10250 1100
@@
 F 0 "C11" H 10865 1146 50  0000 L CNN
 F 1 "100nF" H 10865 1055 50  0000 L CNN
-F 2 "" H 10788 950 50  0001 C CNN
+F 2 "Capacitor_SMD:C_0805_2012Metric" H 10788 950 50  0001 C CNN
 F 3 "~" H 10750 1100 50  0001 C CNN
 	1    10750 1100
@@
 F 0 "C7" H 8365 1146 50  0000 L CNN
 F 1 "100nF" H 8365 1055 50  0000 L CNN
-F 2 "" H 8288 950 50  0001 C CNN
+F 2 "Capacitor_SMD:C_0805_2012Metric" H 8288 950 50  0001 C CNN
 F 3 "~" H 8250 1100 50  0001 C CNN
 	1    8250 1100
@@
 P 1500 4800
 F 0 "C6" H 1615 4846 50  0000 L CNN
-F 1 "C" H 1615 4755 50  0000 L CNN
-F 2 "" H 1538 4650 50  0001 C CNN
+F 1 "100nf" H 1615 4755 50  0000 L CNN
+F 2 "Capacitor_SMD:C_0805_2012Metric" H 1538 4650 50  0001 C CNN
 F 3 "~" H 1500 4800 50  0001 C CNN
 	1    1500 4800
