File: file5F9EC5F3.sch (KiCad schematic (older format))
At the start: 21 parts, among them J4 Conn_ARM_JTAG_SWD_10, SW1 SW_Push, SW2 SW_SPDT, SW3 SW_SPDT, U3 STM32F102R8Tx, Y1 32KHz, Y2 8MHz

Commit message: Preparation for differential routing and small placement corrections.
Connections:
- net OSC_IN_HSE renamed OSC_HSE+
- net OSC_IN_LSE renamed OSC_LSE+
- net OSC_OUT_HSE renamed OSC_HSE-
- net OSC_OUT_LSE renamed OSC_LSE-
- net USB_DATA_MINUS renamed USB_DATA-
- net USB_DATA_PLUS renamed USB_DATA+
Changed lines of the file:
@@
 $EndDescr
 Text Label 5150 3100 2    50   ~ 0
-OSC_IN_HSE
+OSC_HSE+
 Text Label 5150 3200 2    50   ~ 0
-OSC_OUT_HSE
+OSC_HSE-
 Text HLabel 6950 4000 2    50   Output ~ 0
 PELTIER_EN_1
@@
 BT_STATE
 Text HLabel 6950 3000 2    50   BiDi ~ 0
-USB_DATA_MINUS
+USB_DATA-
 Text HLabel 6950 2900 2    50   BiDi ~ 0
-USB_DATA_PLUS
+USB_DATA+
 $Comp
 L Connector:Conn_ARM_JTAG_SWD_10 J4
@@
 Connection ~ 4200 5750
 Text Label 4950 5750 0    50   ~ 0
-OSC_IN_LSE
+OSC_LSE+
 Text Label 4950 6950 0    50   ~ 0
-OSC_IN_HSE
+OSC_HSE+
 Text Label 4950 6050 0    50   ~ 0
-OSC_OUT_LSE
+OSC_LSE-
 Text Label 4950 7250 0    50   ~ 0
-OSC_OUT_HSE
+OSC_HSE-
 $Comp
 L Device:C C9
@@
 	9500 950  9750 950
 Text Label 5150 4900 2    50   ~ 0
-OSC_IN_LSE
+OSC_LSE+
 Text Label 5150 5000 2    50   ~ 0
-OSC_OUT_LSE
+OSC_LSE-
 $Comp
 L MCU_ST_STM32F1:STM32F102R8Tx U3

Commit message: Trackeo
Pobre trackeo parcial. Backup
Connections:
- net +5V is gone; now on net +3V3: SW2.1 (A), SW3.1 (A)
Changed lines of the file:
@@
 	0    1    1    0
-$EndComp
-$Comp
-L power:+5V #PWR031
-U 1 1 5FA25400
-P 2000 6800
-F 0 "#PWR031" H 2000 6650 50  0001 C CNN
-F 1 "+5V" H 2015 6973 50  0000 C CNN
-F 2 "" H 2000 6800 50  0001 C CNN
-F 3 "" H 2000 6800 50  0001 C CNN
-	1    2000 6800
-	1    0    0    -1
 $EndComp
 Text Label 750  7100 2    50   ~ 0
@@
 	1    1350 5950
 	0    1    1    0
-$EndComp
-$Comp
-L power:+5V #PWR043
-U 1 1 5FA3B372
-P 2050 5650
-F 0 "#PWR043" H 2050 5500 50  0001 C CNN
-F 1 "+5V" H 2065 5823 50  0000 C CNN
-F 2 "" H 2050 5650 50  0001 C CNN
-F 3 "" H 2050 5650 50  0001 C CNN
-	1    2050 5650
-	1    0    0    -1
 $EndComp
 Wire Wire Line
@@
 Wire Wire Line
 	6700 3000 6950 3000
+$Comp
+L power:+3.3V #PWR?
+U 1 1 5FB75FE5
+P 2050 5650
+F 0 "#PWR?" H 2050 5500 50  0001 C CNN
+F 1 "+3.3V" H 2065 5823 50  0000 C CNN
+F 2 "" H 2050 5650 50  0001 C CNN
+F 3 "" H 2050 5650 50  0001 C CNN
+	1    2050 5650
+	1    0    0    -1
+$EndComp
+$Comp
+L power:+3.3V #PWR?
+U 1 1 5FB7707A
+P 2000 6800
+F 0 "#PWR?" H 2000 6650 50  0001 C CNN
+F 1 "+3.3V" H 2015 6973 50  0000 C CNN
+F 2 "" H 2000 6800 50  0001 C CNN
+F 3 "" H 2000 6800 50  0001 C CNN
+	1    2000 6800
+	1    0    0    -1
+$EndComp
 $EndSCHEMATC
