File: file5F9F20A5.sch (KiCad schematic (older format))
At the start: 3 parts, among them U4 CR2013-MI2120

Commit message: Finished schematic
Parts:
- BZ1: footprint (none) -> Buzzer_Beeper:Buzzer_Mallory_AST1109MLTRQ
Changed lines of the file:
@@
 $Descr A4 11693 8268
 encoding utf-8
-Sheet 5 7
+Sheet 4 7
 Title ""
 Date ""
@@
 F 0 "BZ1" H 5355 3475 50  0000 C CNN
 F 1 "Buzzer" H 5355 3566 50  0000 C CNN
-F 2 "" V 5325 3900 50  0001 C CNN
+F 2 "Buzzer_Beeper:Buzzer_Mallory_AST1109MLTRQ" V 5325 3900 50  0001 C CNN
 F 3 "~" V 5325 3900 50  0001 C CNN
 	1    5350 3800

Commit message: Added footprints
Parts:
- R3: footprint (none) -> Resistor_SMD:R_0805_2012Metric
Changed lines of the file:
@@
 F 0 "R3" V 5200 3700 50  0000 C CNN
 F 1 "100" V 4984 3700 50  0000 C CNN
-F 2 "" V 5030 3700 50  0001 C CNN
+F 2 "Resistor_SMD:R_0805_2012Metric" V 5030 3700 50  0001 C CNN
 F 3 "~" H 5100 3700 50  0001 C CNN
 	1    5100 3700

Commit message: Placement
Parts:
- added J10, J11: Conn_01x05, Connector_PinSocket_2.54mm:PinSocket_1x05_P2.54mm_Vertical, symbol Connector_Generic:Conn_01x05
- added J12: Conn_01x02, Connector_PinSocket_2.54mm:PinSocket_1x02_P2.54mm_Vertical, symbol Connector_Generic:Conn_01x02
- added J13: Conn_01x09, Connector_PinSocket_2.54mm:PinSocket_1x09_P2.54mm_Vertical, symbol Connector_Generic:Conn_01x09
- added J9: Conn_01x07, Connector_PinSocket_2.54mm:PinSocket_1x07_P2.54mm_Vertical, symbol Connector_Generic:Conn_01x07
Connections:
- net +3V3: now also J12.2 (Pin_2), J9.2 (Pin_2); no longer U4.1 (VCC), U4.8 (LED)
- net GND: now also J12.1 (Pin_1); no longer U4.2 (GND)
- net MISO_IN: now also J10.3 (Pin_3), J9.4 (Pin_4); no longer U4.12 (SD_MISO), U4.9 (MISO)
- net MOSI_IN: now also J10.4 (Pin_4), J9.5 (Pin_5); no longer U4.13 (SD_SCK), U4.6 (MOSI)
- net SCREEN_CS_SPI: now also J9.6 (Pin_6); no longer U4.3 (~CS)
- net SCREEN_D-C_SPI: now also J9.7 (Pin_7); no longer U4.5 (D/~C)
- net SCREEN_RESET: now also J9.1 (Pin_1); no longer U4.4 (RESET)
- net SD_CS_SPI: now also J10.1 (Pin_1); no longer U4.10 (SD_CS)
- net SD_FLASH: now also J10.5 (Pin_5); no longer U4.14 (FLASH_CD)
- net SPI_CLOCK_IN: now also J10.2 (Pin_2), J9.3 (Pin_3); no longer U4.11 (SD_MOSI), U4.7 (SCK)
- new net: J11.5 (Pin_5), U4.10 (SD_CS)
- new net: J11.4 (Pin_4), U4.11 (SD_MOSI)
- new net: J11.3 (Pin_3), U4.12 (SD_MISO)
- new net: J11.2 (Pin_2), U4.13 (SD_SCK)
- new net: J11.1 (Pin_1), U4.14 (FLASH_CD)
- new net PIN_3_ILI: J13.3 (Pin_3), U4.3 (~CS)
- new net PIN_4_ILI: J13.4 (Pin_4), U4.4 (RESET)
- new net PIN_5_ILI: J13.5 (Pin_5), U4.5 (D/~C)
- new net PIN_6_ILI: J13.6 (Pin_6), U4.6 (MOSI)
- new net PIN_7_ILI: J13.7 (Pin_7), U4.7 (SCK)
- new net PIN_8_ILI: J13.8 (Pin_8), U4.8 (LED)
- new net PIN_9_ILI: J13.9 (Pin_9), U4.9 (MISO)
- new net SCREEN_GND_IN: J13.2 (Pin_2), U4.2 (GND)
- new net SCREEN_VCC_IN: J13.1 (Pin_1), U4.1 (VCC)
Other:
- moved on the sheet: BZ1, R3, U4
