File: file5FA096A2.sch (KiCad schematic (older format))
At the start: 3 parts, among them J7 HC 05 Connector, J8 USB_B_Micro, U5 USBLC6-2P6

Commit message: Added footprints
Parts:
- J7, J8: footprint (none) -> Connector_PinHeader_2.54mm:PinHeader_1x06_P2.54mm_Vertical
Changed lines of the file:
@@
 F 0 "J8" H 1107 2067 50  0000 C CNN
 F 1 "USB_B_Micro" H 1107 1976 50  0000 C CNN
-F 2 "" H 1200 1550 50  0001 C CNN
+F 2 "Connector_PinHeader_2.54mm:PinHeader_1x06_P2.54mm_Vertical" H 1200 1550 50  0001 C CNN
 F 3 "~" H 1200 1550 50  0001 C CNN
 	1    1050 1600
@@
 F 0 "J7" H 918 2925 50  0000 C CNN
 F 1 "HC 05 Connector" H 918 3016 50  0000 C CNN
-F 2 "" H 1000 3450 50  0001 C CNN
+F 2 "Connector_PinHeader_2.54mm:PinHeader_1x06_P2.54mm_Vertical" H 1000 3450 50  0001 C CNN
 F 3 "~" H 1000 3450 50  0001 C CNN
 	1    1000 3450

Commit message: Placement
Parts:
- J8: footprint Connector_PinHeader_2.54mm:PinHeader_1x06_P2.54mm_Vertical -> Connector_USB:USB_Micro-B_Molex-105017-0001
Connections:
- wire segments 21 -> 24
Changed lines of the file:
@@
 F 0 "J8" H 1107 2067 50  0000 C CNN
 F 1 "USB_B_Micro" H 1107 1976 50  0000 C CNN
-F 2 "Connector_PinHeader_2.54mm:PinHeader_1x06_P2.54mm_Vertical" H 1200 1550 50  0001 C CNN
+F 2 "Connector_USB:USB_Micro-B_Molex-105017-0001" H 1200 1550 50  0001 C CNN
 F 3 "~" H 1200 1550 50  0001 C CNN
 	1    1050 1600
@@
 U 1 1 5FA0E64B
 P 2750 1650
-F 0 "U5" H 2200 2150 50  0000 C CNN
-F 1 "USBLC6-2P6" H 2400 2050 50  0000 C CNN
+F 0 "U5" V 2300 1500 50  0000 C CNN
+F 1 "USBLC6-2P6" V 2200 1700 50  0000 C CNN
 F 2 "Package_TO_SOT_SMD:SOT-666" H 2750 1150 50  0001 C CNN
 F 3 "https://www.st.com/resource/en/datasheet/usblc6-2.pdf" H 2950 2000 50  0001 C CNN
 	1    2750 1650
-	1    0    0    -1
+	0    1    1    0
 $EndComp
-Wire Wire Line
-	1350 1600 2350 1600
-Wire Wire Line
-	2350 1600 2350 1550
-Wire Wire Line
-	1350 1700 2350 1700
-Wire Wire Line
-	2350 1700 2350 1750
-$Comp
-L power:GND #PWR030
-U 1 1 5FA12A91
-P 2750 2150
-F 0 "#PWR030" H 2750 1900 50  0001 C CNN
-F 1 "GND" H 2755 1977 50  0000 C CNN
-F 2 "" H 2750 2150 50  0001 C CNN
-F 3 "" H 2750 2150 50  0001 C CNN
-	1    2750 2150
-	1    0    0    -1
-$EndComp
-Wire Wire Line
-	2750 2050 2750 2150
-$Comp
-L power:VBUS #PWR029
-U 1 1 5FA132C7
-P 2750 1000
-F 0 "#PWR029" H 2750 850 50  0001 C CNN
-F 1 "VBUS" H 2765 1173 50  0000 C CNN
-F 2 "" H 2750 1000 50  0001 C CNN
-F 3 "" H 2750 1000 50  0001 C CNN
-	1    2750 1000
-	1    0    0    -1
-$EndComp
-Wire Wire Line
-	2750 1000 2750 1250
 NoConn ~ 1350 1800
-Text HLabel 3200 1550 2    50   BiDi ~ 0
+Text HLabel 3250 1250 2    50   BiDi ~ 0
 USB_DATA_PLUS
-Text HLabel 3200 1750 2    50   BiDi ~ 0
+Text HLabel 3250 2050 2    50   BiDi ~ 0
 USB_DATA_MINUS
-Wire Wire Line
-	3150 1550 3200 1550
-Wire Wire Line
-	3150 1750 3200 1750
 $Comp
 L Connector_Generic:Conn_01x06 J7
@@
 Wire Wire Line
 	1650 3150 1200 3150
+Wire Wire Line
+	1350 1600 2100 1600
+Wire Wire Line
+	2100 1600 2100 1250
+Wire Wire Line
+	2100 1250 2650 1250
+Wire Wire Line
+	1350 1700 2100 1700
+Wire Wire Line
+	2100 1700 2100 2050
+Wire Wire Line
+	2100 2050 2650 2050
+$Comp
+L power:VBUS #PWR0102
+U 1 1 5FB251FB
+P 2250 1650
+F 0 "#PWR0102" H 2250 1500 50  0001 C CNN
+F 1 "VBUS" H 2265 1823 50  0000 C CNN
+F 2 "" H 2250 1650 50  0001 C CNN
+F 3 "" H 2250 1650 50  0001 C CNN
+	1    2250 1650
+	1    0    0    -1
+$EndComp
+Wire Wire Line
+	2250 1650 2350 1650
+Wire Wire Line
+	2850 1250 3250 1250
+Wire Wire Line
+	3250 2050 2850 2050
+$Comp
+L power:GND #PWR0103
+U 1 1 5FB28A31
+P 3350 1650
+F 0 "#PWR0103" H 3350 1400 50  0001 C CNN
+F 1 "GND" H 3355 1477 50  0000 C CNN
+F 2 "" H 3350 1650 50  0001 C CNN
+F 3 "" H 3350 1650 50  0001 C CNN
+	1    3350 1650
+	1    0    0    -1
+$EndComp
+Wire Wire Line
+	3350 1700 3350 1650
+Wire Wire Line
+	3350 1650 3150 1650
+Connection ~ 3350 1650
 $EndSCHEMATC

Commit message: Preparation for differential routing and small placement corrections.
Parts:
- J8: footprint Connector_USB:USB_Micro-B_Molex-105017-0001 -> Connector_USB:USB_Micro-B_Wuerth_629105150521
Connections:
- net labels added: D+, D-, USB_DATA+, USB_DATA-
- net labels removed: USB_DATA_MINUS, USB_DATA_PLUS
- wire segments 24 -> 18
Changed lines of the file:
@@
 F 0 "J8" H 1107 2067 50  0000 C CNN
 F 1 "USB_B_Micro" H 1107 1976 50  0000 C CNN
-F 2 "Connector_USB:USB_Micro-B_Molex-105017-0001" H 1200 1550 50  0001 C CNN
+F 2 "Connector_USB:USB_Micro-B_Wuerth_629105150521" H 1200 1550 50  0001 C CNN
 F 3 "~" H 1200 1550 50  0001 C CNN
 	1    1050 1600
@@
 NoConn ~ 1350 1800
 Text HLabel 3250 1250 2    50   BiDi ~ 0
-USB_DATA_PLUS
+USB_DATA+
 Text HLabel 3250 2050 2    50   BiDi ~ 0
-USB_DATA_MINUS
+USB_DATA-
 $Comp
 L Connector_Generic:Conn_01x06 J7
@@
 Wire Wire Line
 	1650 3150 1200 3150
-Wire Wire Line
-	1350 1600 2100 1600
-Wire Wire Line
-	2100 1600 2100 1250
-Wire Wire Line
-	2100 1250 2650 1250
-Wire Wire Line
-	1350 1700 2100 1700
-Wire Wire Line
-	2100 1700 2100 2050
-Wire Wire Line
-	2100 2050 2650 2050
 $Comp
 L power:VBUS #PWR0102
@@
 	3350 1650 3150 1650
 Connection ~ 3350 1650
+Text Label 1350 1600 0    50   ~ 0
+D+
+Text Label 1350 1700 0    50   ~ 0
+D-
+Text Label 2650 2050 0    50   ~ 0
+D-
+Text Label 2650 1250 0    50   ~ 0
+D+
 $EndSCHEMATC
