File: _autosave-file5F9EC5F3.sch (KiCad schematic (older format))
At the start: 21 parts, among them J4 Conn_ARM_JTAG_SWD_10, SW1 SW_Push, SW2 SW_SPDT, SW3 SW_SPDT, U3 STM32F102R8Tx, Y1 32KHz, Y2 8MHz

Commit message: Trackeo
Pobre trackeo parcial. Backup
Connections:
- net +5V is gone; now on net +3V3: SW2.1 (A), SW3.1 (A)
- net THERMISTOR_IN_1: now also U3.25 (PC5); no longer U3.24 (PC4)
- net THERMISTOR_IN_2: now also U3.24 (PC4); no longer U3.25 (PC5)
Changed lines of the file:
@@
 BUZZER_PWM_IN
 Text HLabel 5150 3900 0    50   Input ~ 0
+THERMISTOR_IN_2
+Text HLabel 5150 4000 0    50   Input ~ 0
 THERMISTOR_IN_1
-Text HLabel 5150 4000 0    50   Input ~ 0
-THERMISTOR_IN_2
 Text HLabel 6950 2100 2    50   Input ~ 0
 BT_STATE
@@
 	0    1    1    0
 $EndComp
-$Comp
-L power:+5V #PWR031
-U 1 1 5FA25400
-P 2000 6800
-F 0 "#PWR031" H 2000 6650 50  0001 C CNN
-F 1 "+5V" H 2015 6973 50  0000 C CNN
-F 2 "" H 2000 6800 50  0001 C CNN
-F 3 "" H 2000 6800 50  0001 C CNN
-	1    2000 6800
-	1    0    0    -1
-$EndComp
 Text Label 750  7100 2    50   ~ 0
 BOOT1
@@
 	1    1350 5950
 	0    1    1    0
-$EndComp
-$Comp
-L power:+5V #PWR043
-U 1 1 5FA3B372
-P 2050 5650
-F 0 "#PWR043" H 2050 5500 50  0001 C CNN
-F 1 "+5V" H 2065 5823 50  0000 C CNN
-F 2 "" H 2050 5650 50  0001 C CNN
-F 3 "" H 2050 5650 50  0001 C CNN
-	1    2050 5650
-	1    0    0    -1
 $EndComp
 Wire Wire Line
@@
 Wire Wire Line
 	6700 3000 6950 3000
+$Comp
+L power:+3.3V #PWR0106
+U 1 1 5FB75FE5
+P 2050 5650
+F 0 "#PWR0106" H 2050 5500 50  0001 C CNN
+F 1 "+3.3V" H 2065 5823 50  0000 C CNN
+F 2 "" H 2050 5650 50  0001 C CNN
+F 3 "" H 2050 5650 50  0001 C CNN
+	1    2050 5650
+	1    0    0    -1
+$EndComp
+$Comp
+L power:+3.3V #PWR0107
+U 1 1 5FB7707A
+P 2000 6800
+F 0 "#PWR0107" H 2000 6650 50  0001 C CNN
+F 1 "+3.3V" H 2015 6973 50  0000 C CNN
+F 2 "" H 2000 6800 50  0001 C CNN
+F 3 "" H 2000 6800 50  0001 C CNN
+	1    2000 6800
+	1    0    0    -1
+$EndComp
 $EndSCHEMATC
